File: pcb/dizzy40.kicad_pcb (KiCad board)
At the start: 2 copper layers, 229 x 80 mm, 55 parts

Commit message: diode positioning done
Parts:
- removed MX1, MX10, MX11, MX13, MX14, MX15, MX16, MX17, MX18, MX19, MX2, MX20, MX21, MX24, MX25, MX26, MX27, MX28, MX29, MX3, MX30, MX31, MX32, MX35, MX4, MX41, MX43, MX5, MX50, MX51, MX52, MX54, MX6, MX7, MX8, MX9: MX-NoLED, MX_Only:MXOnly-1U-NoLED
- removed MX12, MX33, MX34, MX36, MX40, MX42, MX49, MX53: MX-NoLED, MX_Only:MXOnly-1.25U-NoLED
- removed MX22, MX23: MX-NoLED, MX_Only:MXOnly-1.75U-NoLED
- removed MX37: MX-NoLED, MX_Only:MXOnly-3U-ReversedStabilizers-NoLED
- removed MX39: MX-NoLED, MX_Only:MXOnly-2U-ReversedStabilizers-NoLED
- removed MX44, MX47: MX-NoLED, MX_Only:MXOnly-2.75U-ReversedStabilizers-NoLED
- removed MX45, MX46: MX-NoLED, MX_Only:MXOnly-2.25U-ReversedStabilizers-NoLED
- removed MX48, MX55: MX-NoLED, MX_Only:MXOnly-1.5U-NoLED
- removed USB1: USB_C_Receptacle_USB2.0, Connector_USB:USB_C_Receptacle_HRO_TYPE-C-31-M-12
- added C1: 10u, Capacitor_SMD:C_0805_2012Metric, B.Cu at (210.6, 77.8)
- added C10: 1u, Capacitor_SMD:C_0805_2012Metric, B.Cu at (231.2, 81.8)
- added C11: 100n, Capacitor_SMD:C_0805_2012Metric, B.Cu at (222.3, 77.8)
- added C12: 100n, Capacitor_SMD:C_0805_2012Metric, B.Cu at (220.3, 77.8)
- added C13: 100n, Capacitor_SMD:C_0805_2012Metric, B.Cu at (224.3, 77.8)
- added C14: 100n, Capacitor_SMD:C_0805_2012Metric, B.Cu at (226.3, 77.8)
- added C17: 10u, Capacitor_SMD:C_0805_2012Metric, B.Cu at (216.3, 77.8)
- added C2: 22pf, Capacitor_SMD:C_0805_2012Metric, B.Cu at (234.3, 99.5)
- added C3: 22pf, Capacitor_SMD:C_0805_2012Metric, B.Cu at (229.9, 95.1)
- added C4: 10u, Capacitor_SMD:C_0805_2012Metric, B.Cu at (218.3, 77.8)
- added C5: 100n, Capacitor_SMD:C_0805_2012Metric, B.Cu at (249.6, 80.2)
- added C6: 100n, Capacitor_SMD:C_0805_2012Metric, B.Cu at (190.5, 26.2)
- added C7: 100n, Capacitor_SMD:C_0805_2012Metric, B.Cu at (189.1, 21.4)
- added C8: 1u, Capacitor_SMD:C_0805_2012Metric, B.Cu at (193.8, 21.4)
- added C9: 100n, Capacitor_SMD:C_0805_2012Metric, B.Cu at (228.4, 77.8)
- added D17: BAV70, Package_TO_SOT_SMD:SOT-23, B.Cu at (58.6, 73.2)
- added D18: BAV70, Package_TO_SOT_SMD:SOT-23, B.Cu at (58.3, 76.8)
- added D19: BAV70, Package_TO_SOT_SMD:SOT-23, B.Cu at (58.1, 80.3)
- added D20: BAV70, Package_TO_SOT_SMD:SOT-23, B.Cu at (192.9, 95.7)
- added D21: BAV70, Package_TO_SOT_SMD:SOT-23, B.Cu at (201.9, 63.1)
- added D22: BAV70, Package_TO_SOT_SMD:SOT-23, B.Cu at (193.7, 99.3)
- added D23: BAV70, Package_TO_SOT_SMD:SOT-23, B.Cu at (57.9, 91.1)
- added D24: BAV70, Package_TO_SOT_SMD:SOT-23, B.Cu at (57.9, 87.5)
- added D25: BAV70, Package_TO_SOT_SMD:SOT-23, B.Cu at (57.9, 83.9)
- added D26: BAV70, Package_TO_SOT_SMD:SOT-23, B.Cu at (192.5, 92.1)
- added D27: BAV70, Package_TO_SOT_SMD:SOT-23, B.Cu at (195.7, 105.0)
- added D28: BAV70, Package_TO_SOT_SMD:SOT-23, B.Cu at (200.7, 113.3)
- added D29: BAV70, Package_TO_SOT_SMD:SOT-23, B.Cu at (58.0, 94.7)
- added D30: BAV70, Package_TO_SOT_SMD:SOT-23, B.Cu at (58.1, 98.2)
- added D31: BAV70, Package_TO_SOT_SMD:SOT-23, B.Cu at (58.3, 101.8)
- added D32: BAV70, Package_TO_SOT_SMD:SOT-23, B.Cu at (205.8, 118.7)
- added D33: BAV70, Package_TO_SOT_SMD:SOT-23, B.Cu at (198.5, 110.3)
- added D34: BAV70, Package_TO_SOT_SMD:SOT-23, B.Cu at (203.1, 116.1)
- added D35: BAV70, Package_TO_SOT_SMD:SOT-23, B.Cu at (60.0, 116.1)
- added D36: BAV70, Package_TO_SOT_SMD:SOT-23, B.Cu at (59.5, 112.5)
- added D37: BAV70, Package_TO_SOT_SMD:SOT-23, B.Cu at (59.1, 109.0)
- added D38: BAV70, Package_TO_SOT_SMD:SOT-23, B.Cu at (58.6, 105.4)
- added D39: BAV70, Package_TO_SOT_SMD:SOT-23, B.Cu at (214.8, 124.7)
- added ENC1: RotaryEncoder_Switch, Keebio-Parts:RotaryEncoder_Alps_EC11E-Switch_Vertical_H20mm, B.Cu at (42.9, 69.9)
- added ENC2: RotaryEncoder_Switch, Keebio-Parts:RotaryEncoder_Alps_EC11E-Switch_Vertical_H20mm, B.Cu at (142.9, 127.0)
- added F0: polyfuse, Fuse:Fuse_1206_3216Metric, B.Cu at (145.5, 69.9)
- added J0: USB_C_Receptacle_USB2.0, Connector_USB:USB_C_Receptacle_HRO_TYPE-C-31-M-12, B.Cu at (147.7, 59.5)
- added J1: BREAKOUT, Connector_PinSocket_2.54mm:PinSocket_1x05_P2.54mm_Vertical, B.Cu at (157.1, 32.9)
- added J2: Conn_01x03_Male, Connector_PinSocket_2.54mm:PinSocket_1x03_P2.54mm_Vertical, B.Cu at (129.8, 21.0)
- added J3: 3x Breakout | additional pins, Connector_PinSocket_2.54mm:PinSocket_1x03_P2.54mm_Vertical, B.Cu at (152.5, 32.9)
- added J4: Breakout 1.1v, Connector_PinSocket_2.54mm:PinSocket_1x02_P2.54mm_Vertical, B.Cu at (152.5, 42.6)
- added K1: KEYSW, marbastlib-mx:SW_MX_1u, F.Cu at (42.9, 69.9)
- added K10: KEYSW, marbastlib-mx:SW_MX_1u, F.Cu at (214.3, 69.9)
- added K11: KEYSW, marbastlib-mx:SW_MX_1u, F.Cu at (233.4, 69.9)
- added K12: KEYSW, marbastlib-mx:SW_MX_1u, F.Cu at (45.3, 88.9)
- added K13: KEYSW, marbastlib-mx:SW_MX_1u, F.Cu at (66.7, 88.9)
- added K14: KEYSW, marbastlib-mx:SW_MX_1u, F.Cu at (85.7, 88.9)
- added K15: KEYSW, marbastlib-mx:SW_MX_1u, F.Cu at (104.8, 88.9)
- added K16: KEYSW, marbastlib-mx:SW_MX_1u, F.Cu at (123.8, 88.9)
- added K17: KEYSW, marbastlib-mx:SW_MX_1u, F.Cu at (142.9, 88.9)
- added K18: KEYSW, marbastlib-mx:SW_MX_1u, F.Cu at (161.9, 88.9)
- added K19: KEYSW, marbastlib-mx:SW_MX_1u, F.Cu at (181.0, 88.9)
- added K2: KEYSW, marbastlib-mx:SW_MX_1u, F.Cu at (61.9, 69.9)
- added K20: KEYSW, marbastlib-mx:SW_MX_1u, F.Cu at (200.0, 88.9)
- added K21: KEYSW, marbastlib-mx:SW_MX_1u, F.Cu at (219.1, 88.9)
- added K22: KEYSW, marbastlib-mx:SW_MX_1u, F.Cu at (245.3, 88.9)
- added K23: KEYSW, marbastlib-mx:SW_MX_1u, F.Cu at (50.0, 108.0)
- added K24: KEYSW, marbastlib-mx:SW_MX_1u, F.Cu at (76.2, 108.0)
- added K25: KEYSW, marbastlib-mx:SW_MX_1u, F.Cu at (95.3, 108.0)
- added K26: KEYSW, marbastlib-mx:SW_MX_1u, F.Cu at (114.3, 108.0)
- added K27: KEYSW, marbastlib-mx:SW_MX_1u, F.Cu at (133.4, 108.0)
- added K28: KEYSW, marbastlib-mx:SW_MX_1u, F.Cu at (152.4, 108.0)
- added K29: KEYSW, marbastlib-mx:SW_MX_1u, F.Cu at (171.5, 108.0)
- added K3: KEYSW, marbastlib-mx:SW_MX_1u, F.Cu at (81.0, 69.9)
- added K30: KEYSW, marbastlib-mx:SW_MX_1u, F.Cu at (190.5, 108.0)
- added K31: KEYSW, marbastlib-mx:SW_MX_1u, F.Cu at (209.6, 108.0)
- added K32: KEYSW, marbastlib-mx:SW_MX_1u, F.Cu at (228.6, 108.0)
- added K33: KEYSW, marbastlib-mx:SW_MX_1u, F.Cu at (250.0, 108.0)
- added K34: KEYSW, marbastlib-mx:SW_MX_1u, F.Cu at (45.3, 127.0)
- added K35: KEYSW, marbastlib-mx:SW_MX_1u, F.Cu at (66.7, 127.0)
- added K36: KEYSW, marbastlib-mx:SW_MX_1u, F.Cu at (90.5, 127.0)
- added K37: KEYSW, marbastlib-mx:SW_MX_1u, F.Cu at (116.7, 127.0)
- added K38: KEYSW, marbastlib-mx:SW_MX_1u, F.Cu at (142.9, 127.0)
- added K39: KEYSW, marbastlib-mx:SW_MX_1u, F.Cu at (169.1, 127.0)
- added K4: KEYSW, marbastlib-mx:SW_MX_1u, F.Cu at (100.0, 69.9)
- added K40: KEYSW, marbastlib-mx:SW_MX_1u, F.Cu at (207.2, 127.0)
- added K41: KEYSW, marbastlib-mx:SW_MX_1u, F.Cu at (226.2, 127.0)
- added K42: KEYSW, marbastlib-mx:SW_MX_1u, F.Cu at (250.0, 127.0)
- added K45: KEYSW, marbastlib-mx:SW_MX_1u, F.Cu at (128.6, 127.0)
- added K46: KEYSW, marbastlib-mx:SW_MX_1u, F.Cu at (121.5, 127.0)
- added K49: KEYSW, marbastlib-mx:SW_MX_1u, F.Cu at (247.7, 127.0)
- added K5: KEYSW, marbastlib-mx:SW_MX_1u, F.Cu at (119.1, 69.9)
- added K50: KEYSW, marbastlib-mx:SW_MX_1u, F.Cu at (223.9, 127.0)
- added K51: KEYSW, marbastlib-mx:SW_MX_1u, F.Cu at (47.6, 127.0)
- added K52: KEYSW, marbastlib-mx:SW_MX_1u, F.Cu at (71.5, 127.0)
- added K53: KEYSW, marbastlib-mx:SW_MX_1u, F.Cu at (88.1, 127.0)
- added K54: KEYSW, marbastlib-mx:SW_MX_1u, F.Cu at (126.2, 127.0)
- added K55: KEYSW, marbastlib-mx:SW_MX_1u, F.Cu at (173.8, 127.0)
- added K56: KEYSW, marbastlib-mx:SW_MX_1u, F.Cu at (204.8, 127.0)
- added K57: KEYSW, marbastlib-mx:SW_MX_1u, F.Cu at (176.2, 127.0)
- added K58: KEYSW, marbastlib-mx:SW_MX_1u, F.Cu at (228.6, 127.0)
- added K59: KEYSW, marbastlib-mx:SW_MX_1u, F.Cu at (252.4, 69.9)
- added K6: KEYSW, marbastlib-mx:SW_MX_1u, F.Cu at (138.1, 69.9)
- added K7: KEYSW, marbastlib-mx:SW_MX_1u, F.Cu at (157.2, 69.9)
- added K8: KEYSW, marbastlib-mx:SW_MX_1u, F.Cu at (176.2, 69.9)
- added K9: KEYSW, marbastlib-mx:SW_MX_1u, F.Cu at (195.3, 69.9)
- added R1: 1k, Resistor_SMD:R_0805_2012Metric, B.Cu at (251.7, 80.2)
- added R3: 27, Resistor_SMD:R_0805_2012Metric, B.Cu at (153.1, 75.0)
- added R4: 27, Resistor_SMD:R_0805_2012Metric, B.Cu at (149.6, 72.5)
- added R5: 1k, Resistor_SMD:R_0805_2012Metric, B.Cu at (228.4, 93.7)
- added R6: 5.1k, Resistor_SMD:R_0805_2012Metric, B.Cu at (154.7, 61.9)
- added R7: 5.1k, Resistor_SMD:R_0805_2012Metric, B.Cu at (140.6, 61.9)
- added R8: 10k, Resistor_SMD:R_0805_2012Metric, B.Cu at (274.6, 99.6)
- added REF**: STAB_MX_P_2u, marbastlib-mx:STAB_MX_P_2u, F.Cu at (173.8, 127.0)
- added REF**: STAB_MX_P_2u, marbastlib-mx:STAB_MX_P_2u, B.Cu at (169.1, 127.0)
- added REF**: STAB_MX_P_2u, marbastlib-mx:STAB_MX_P_2u, B.Cu at (176.2, 127.0)
- added REF**: STAB_MX_P_2u, marbastlib-mx:STAB_MX_P_2u, B.Cu at (126.2, 127.0)
- added REF**: STAB_MX_P_2u, marbastlib-mx:STAB_MX_P_2u, B.Cu at (121.5, 127.0)
- added RGB1: WS2812B, kbd:LED_WS2812B-PLCC4, B.Cu at (199.7, 79.4)
- added RGB2: WS2812B, kbd:LED_WS2812B-PLCC4, B.Cu at (186.7, 98.4)
- added RGB3: WS2812B, kbd:LED_WS2812B-PLCC4, B.Cu at (173.7, 79.4)
- added RGB4: WS2812B, kbd:LED_WS2812B-PLCC4, B.Cu at (160.7, 98.4)
- added RGB5: WS2812B, kbd:LED_WS2812B-PLCC4, B.Cu at (147.7, 79.2)
- added RGB6: WS2812B, kbd:LED_WS2812B-PLCC4, B.Cu at (134.7, 98.4)
- added RGB7: WS2812B, kbd:LED_WS2812B-PLCC4, B.Cu at (121.7, 79.4)
- added RGB8: WS2812B, kbd:LED_WS2812B-PLCC4, B.Cu at (108.7, 98.4)
- added RGB9: WS2812B, kbd:LED_WS2812B-PLCC4, B.Cu at (95.7, 79.4)
- added SW0: RESET, Keebio-Parts:SW_SPST_TL3342, B.Cu at (261.1, 87.8)
- added SW2: RESET, Keebio-Parts:SW_SPST_TL3342, B.Cu at (267.9, 100.1)
- added U2: W25Q128JVS, Package_SO:SOIC-8_5.23x5.23mm_P1.27mm, B.Cu at (242.9, 79.0)
- added U3: RP2040, RP2040:RP2040-QFN-56, B.Cu at (232.2, 88.9)
- added U4: XC6206P Smaller footprint, less mA ~.5, Package_TO_SOT_SMD:SOT-23, B.Cu at (213.5, 77.8)
- added U44: SRV05-4, Package_TO_SOT_SMD:SOT-23-6, B.Cu at (148.7, 69.3)
- added Y0: 12MHZ Crystal, Crystal:Crystal_SMD_3225-4Pin_3.2x2.5mm, B.Cu at (232.1, 97.3)
Routing:
- net GND: track 0.00 -> 402.1 mm, vias 0 -> 5
- net +5V: track 0.00 -> 307.6 mm, vias 0 -> 2
- net ROW2: track 0.00 -> 209.7 mm, vias 0 -> 3
- net Net-(D38-A-Pad1): track 0.00 -> 186.2 mm
- net ROW3: track 0.00 -> 181.0 mm
- net Net-(D38-A-Pad2): track 0.00 -> 165.1 mm
- net Net-(D37-A-Pad1): track 0.00 -> 128.9 mm
- net COL7: track 0.00 -> 118.1 mm
- net Net-(D31-A-Pad2): track 0.00 -> 116.0 mm
- net COL8: track 0.00 -> 110.6 mm
- net COL5: track 0.00 -> 107.9 mm
- net COL6: track 0.00 -> 106.5 mm
- net Net-(D20-A-Pad1): track 0.00 -> 105.5 mm
- net Net-(D26-A-Pad2): track 0.00 -> 101.1 mm
- net COL3: track 0.00 -> 98.4 mm
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Other:
- board text removed: "Dizzy40 rev.1 keyboards.elmo.space"

Commit message: positions reset buttons, routing
Parts:
- moved J1 73.3 mm to (212.1, 81.4), turned to -90 degrees
- moved R8 28.0 mm to (252.6, 82.3), turned to -80 degrees
- moved SW2 19.2 mm to (257.0, 84.2), turned to 100 degrees
- moved R1 15.3 mm to (252.6, 95.5), turned to -100 degrees
- moved SW0 7.15 mm to (257.0, 93.6), turned to 80 degrees
- moved C2 3.75 mm to (230.7, 98.7), turned to -135 degrees
- moved Y0 3.75 mm to (228.4, 96.4)
- moved C3 3.75 mm to (226.2, 94.2), turned to -135 degrees
- moved R5 3.75 mm to (224.8, 92.8), turned to -135 degrees
- moved R3 2.53 mm to (153.0, 72.5)
- moved C5 0.21 mm to (249.6, 79.9)
- moved U2 0.20 mm to (242.9, 78.8)
Routing:
- net ENC_ESC_R: track 0.00 -> 117.6 mm, vias 0 -> 3
- net ENC_ESC_L: track 0.00 -> 115.4 mm, vias 0 -> 3
- net ROW0: track 7.40 -> 119.6 mm, vias 0 -> 3
- net ROW1: track 23.6 -> 122.1 mm
- net GND: track 402.1 -> 488.5 mm, vias 5 -> 7
- net +3V3: track 36.0 -> 95.5 mm
- net /MCU/QSPI_SS: track 8.96 -> 35.5 mm, vias 0 -> 2
- net +5V: track 307.6 -> 287.5 mm
- net Net-(U3-USB_DP): track 85.9 -> 66.7 mm
- net Net-(U3-USB_DM): track 88.2 -> 70.4 mm
- net COL0: track 89.3 -> 106.6 mm
- net /MCU/RUN: track 0.00 -> 13.6 mm
- net /MCU/XIN: track 0.00 -> 10.2 mm
- net /MCU/~{USB_BOOT}: track 0.00 -> 8.85 mm
- net /MCU/XOUT: track 0.00 -> 7.51 mm
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
Commit message: finalized routing, placement of components
Parts:
- removed REF** (x5): STAB_MX_P_2u, marbastlib-mx:STAB_MX_P_2u
- added J5: Screw_Terminal_01x02, marbastlib-mx:STAB_MX_P_2u, F.Cu at (126.2, 127.0)
- added J6: Screw_Terminal_01x02, marbastlib-mx:STAB_MX_P_2u, F.Cu at (169.1, 127.0)
- added J7: Screw_Terminal_01x02, marbastlib-mx:STAB_MX_P_2u, F.Cu at (173.8, 127.0)
- added J8: Screw_Terminal_01x02, marbastlib-mx:STAB_MX_P_2u, F.Cu at (176.2, 127.0)
- J3: value 3x Breakout | additional pins -> Screw_Terminal_01x02; footprint Connector_PinSocket_2.54mm:PinSocket_1x03_P2.54mm_Vertical -> marbastlib-mx:STAB_MX_P_2u; moved to F.Cu
- moved J3 99.1 mm to (121.5, 127.0)
- moved J2 98.0 mm to (212.1, 74.3), turned to -90 degrees
- moved J4 86.4 mm to (219.7, 96.9), turned to 90 degrees
- moved C7 78.5 mm to (210.7, 96.9), turned to -90 degrees
- moved C8 78.3 mm to (214.8, 96.9), turned to -90 degrees
- moved C6 74.1 mm to (212.8, 96.9), turned to -90 degrees
- moved R3 4.21 mm to (148.8, 72.5)
- moved R4 2.15 mm to (148.8, 70.5)
- moved F0 1.59 mm to (145.5, 68.3)
- moved U44 1.59 mm to (148.8, 67.7)
- turned C11 to -90 degrees
- turned C12 to -90 degrees
- turned C13 to -90 degrees
- turned C14 to -90 degrees
- turned C17 to -90 degrees
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Connections:
- D17 pad 1: Net-(D17-A-Pad1) -> ENC_ROW_TOP
- D37 pad 2: Net-(D37-A-Pad2) -> ENC_ROW_MID
- ENC1 pad S1: unconnected-(ENC1-PadS1) -> ENC_ROW_TOP
- ENC1 pad S2: unconnected-(ENC1-PadS2) -> COL0
- ENC2 pad S1: unconnected-(ENC2-PadS1) -> ENC_ROW_MID
- ENC2 pad S2: unconnected-(ENC2-PadS2) -> COL4
- J1 pad 1: /MCU/RUN -> GND
- J1 pad 3: GND -> /MCU/RUN
- J3 pad 1: unconnected-(J3-Pin_1-Pad1) -> GND
- J3 pad 2: unconnected-(J3-Pin_2-Pad2) -> GND
- K1 pad 1: Net-(D17-A-Pad1) -> ENC_ROW_TOP
- K38 pad 1: Net-(D37-A-Pad2) -> ENC_ROW_MID
- K59 pad 1: unconnected-(K59-Pad1) -> COL11
- U3 pad 11: col0 -> COL2
- U3 pad 12: col1 -> COL3
- U3 pad 13: col2 -> COL4
- U3 pad 14: col3 -> COL5
- U3 pad 15: col4 -> COL6
- U3 pad 16: col5 -> COL7
- U3 pad 17: col6 -> COL8
- U3 pad 18: col7 -> COL9
- U3 pad 2: ENC_SPC_L -> ROW3
- U3 pad 27: col8 -> unconnected-(U3-GPIO16-Pad27)
- U3 pad 28: col9 -> ENC_ESC_R
- U3 pad 29: col10 -> ENC_ESC_L
- U3 pad 3: ENC_SPC_R -> RGB
- U3 pad 30: unconnected-(U3-GPIO19-Pad30) -> ROW0
- U3 pad 35: unconnected-(U3-GPIO23-Pad35) -> ROW1
- U3 pad 36: unconnected-(U3-GPIO24-Pad36) -> LED_GLOW
- U3 pad 37: unconnected-(U3-GPIO25-Pad37) -> COL11
- U3 pad 4: ENC_ESC_L -> ROW2
- U3 pad 5: ENC_ESC_R -> COL10
- U3 pad 6: row0 -> ENC_SPC_L
- U3 pad 7: row1 -> ENC_SPC_R
- U3 pad 8: row2 -> COL0
- U3 pad 9: row3 -> COL1
Routing:
- net GND: track 488.5 -> 872.4 mm, vias 7 -> 30
- net COL1: track 92.1 -> 327.1 mm, vias 0 -> 1
- net COL0: track 106.6 -> 329.8 mm, vias 0 -> 1
- net COL2: track 95.4 -> 285.5 mm, vias 0 -> 1
- net ROW0: track 119.6 -> 303.3 mm, vias 3 -> 7
- net COL3: track 98.4 -> 280.3 mm, vias 0 -> 1
- net ROW1: track 122.1 -> 286.9 mm, vias 1 -> 4
- net ENC_SPC_R: track 0.00 -> 148.3 mm, vias 0 -> 1
- net ENC_SPC_L: track 0.00 -> 146.8 mm, vias 0 -> 1
- net COL4: track 83.6 -> 224.1 mm, vias 0 -> 1
- net RGB: track 0.00 -> 129.6 mm, vias 0 -> 3
- net COL5: track 107.9 -> 237.1 mm, vias 0 -> 1
- net ENC_ROW_MID: track 0.00 -> 101.7 mm
- net Net-(D37-A-Pad2): track 95.7 -> 0.00 mm
- net ENC_ESC_R: track 117.6 -> 212.0 mm, vias 3 -> 5
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- added copper zone on B.Cu, net GND
- added copper zone on F.Cu, net GND
Other:
- board text removed: "|"
